File: MiSTerDualshock.sch (EAGLE design)
At the start: 21 parts, among them K1 692121030100

Commit message: Added pull-up resistor to DAT line
Parts:
- added R1: 10K, resistor:R-US_0207/10
Connections:
- net 3V3: now also R1.2
- net DAT: now also R1.1
Changed lines of the file:
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@@
 <part name="J1" library="con-jack" deviceset="JACK-PLUG" device="1"/>
 <part name="JP1" library="pinhead" deviceset="PINHD-1X3" device=""/>
+<part name="R1" library="resistor" deviceset="R-US_" device="0207/10" value="10K"/>
 </parts>
 <sheets>
@@
 <instance part="J1" gate="G$1" x="144.78" y="50.8"/>
 <instance part="JP1" gate="A" x="91.44" y="58.42"/>
+<instance part="R1" gate="G$1" x="187.96" y="53.34" rot="R90"/>
 </instances>
 <busses>
@@
 <wire x1="88.9" y1="60.96" x2="78.74" y2="60.96" width="0.1524" layer="91"/>
 <label x="78.74" y="60.96" size="1.778" layer="95"/>
+</segment>
+<segment>
+<pinref part="R1" gate="G$1" pin="2"/>
+<wire x1="187.96" y1="58.42" x2="187.96" y2="63.5" width="0.1524" layer="91"/>
+<label x="187.96" y="60.96" size="1.778" layer="95" rot="R90"/>
 </segment>
 </net>
@@
 <label x="167.64" y="7.62" size="1.778" layer="95"/>
 </segment>
+<segment>
+<pinref part="R1" gate="G$1" pin="1"/>
+<wire x1="187.96" y1="48.26" x2="187.96" y2="43.18" width="0.1524" layer="91"/>
+<label x="187.96" y="43.18" size="1.778" layer="95" rot="R90"/>
+</segment>
 </net>

Commit message: Version 1.2
Parts:
- added R2, R3, R4, R5: 10K, resistor:R-US_0207/10
Connections:
- net 3V3: now also R2.2, R3.2, R4.2, R5.2
- net ATT1: now also R2.1
- net ATT2: now also R5.1
- net CLK: now also R1.1
- net CMD: now also R4.1
- net DAT: now also R3.1; no longer R1.1
Changed lines of the file:
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@@
 <part name="JP1" library="pinhead" deviceset="PINHD-1X3" device=""/>
 <part name="R1" library="resistor" deviceset="R-US_" device="0207/10" value="10K"/>
+<part name="R2" library="resistor" deviceset="R-US_" device="0207/10" value="10K"/>
+<part name="R3" library="resistor" deviceset="R-US_" device="0207/10" value="10K"/>
+<part name="R4" library="resistor" deviceset="R-US_" device="0207/10" value="10K"/>
+<part name="R5" library="resistor" deviceset="R-US_" device="0207/10" value="10K"/>
 </parts>
 <sheets>
@@
 <instance part="JP1" gate="A" x="91.44" y="58.42"/>
 <instance part="R1" gate="G$1" x="187.96" y="53.34" rot="R90"/>
+<instance part="R2" gate="G$1" x="198.12" y="53.34" rot="R90"/>
+<instance part="R3" gate="G$1" x="167.64" y="53.34" rot="R90"/>
+<instance part="R4" gate="G$1" x="177.8" y="53.34" rot="R90"/>
+<instance part="R5" gate="G$1" x="208.28" y="53.34" rot="R90"/>
 </instances>
 <busses>
@@
 <label x="167.64" y="10.16" size="1.778" layer="95"/>
 </segment>
+<segment>
+<pinref part="R1" gate="G$1" pin="1"/>
+<wire x1="187.96" y1="48.26" x2="187.96" y2="43.18" width="0.1524" layer="91"/>
+<label x="187.96" y="43.18" size="1.778" layer="95" rot="R90"/>
+</segment>
 </net>
 <net name="3V3" class="0">
@@
 <wire x1="187.96" y1="58.42" x2="187.96" y2="63.5" width="0.1524" layer="91"/>
 <label x="187.96" y="60.96" size="1.778" layer="95" rot="R90"/>
+</segment>
+<segment>
+<pinref part="R2" gate="G$1" pin="2"/>
+<wire x1="198.12" y1="58.42" x2="198.12" y2="63.5" width="0.1524" layer="91"/>
+<label x="198.12" y="60.96" size="1.778" layer="95" rot="R90"/>
+</segment>
+<segment>
+<pinref part="R3" gate="G$1" pin="2"/>
+<wire x1="167.64" y1="58.42" x2="167.64" y2="63.5" width="0.1524" layer="91"/>
+<label x="167.64" y="60.96" size="1.778" layer="95" rot="R90"/>
+</segment>
+<segment>
+<pinref part="R4" gate="G$1" pin="2"/>
+<wire x1="177.8" y1="58.42" x2="177.8" y2="63.5" width="0.1524" layer="91"/>
+<label x="177.8" y="60.96" size="1.778" layer="95" rot="R90"/>
+</segment>
+<segment>
+<pinref part="R5" gate="G$1" pin="2"/>
+<wire x1="208.28" y1="58.42" x2="208.28" y2="63.5" width="0.1524" layer="91"/>
+<label x="208.28" y="60.96" size="1.778" layer="95" rot="R90"/>
 </segment>
 </net>
@@
 <label x="167.64" y="17.78" size="1.778" layer="95"/>
 </segment>
+<segment>
+<pinref part="R4" gate="G$1" pin="1"/>
+<wire x1="177.8" y1="48.26" x2="177.8" y2="43.18" width="0.1524" layer="91"/>
+<label x="177.8" y="43.18" size="1.778" layer="95" rot="R90"/>
+</segment>
 </net>
 <net name="DAT" class="0">
@@
 </segment>
 <segment>
-<pinref part="R1" gate="G$1" pin="1"/>
-<wire x1="187.96" y1="48.26" x2="187.96" y2="43.18" width="0.1524" layer="91"/>
-<label x="187.96" y="43.18" size="1.778" layer="95" rot="R90"/>
+<pinref part="R3" gate="G$1" pin="1"/>
+<wire x1="167.64" y1="48.26" x2="167.64" y2="43.18" width="0.1524" layer="91"/>
+<label x="167.64" y="43.18" size="1.778" layer="95" rot="R90"/>
 </segment>
 </net>
@@
 <label x="167.64" y="25.4" size="1.778" layer="95"/>
 </segment>
+<segment>
+<pinref part="R2" gate="G$1" pin="1"/>
+<wire x1="198.12" y1="48.26" x2="198.12" y2="43.18" width="0.1524" layer="91"/>
+<label x="198.12" y="43.18" size="1.778" layer="95" rot="R90"/>
+</segment>
 </net>
 <net name="ATT2" class="0">
@@
 <label x="167.64" y="22.86" size="1.778" layer="95"/>
 </segment>
-</net>
+<segment>
+<pinref part="R5" gate="G$1" pin="1"/>
+<wire x1="208.28" y1="48.26" x2="208.28" y2="43.18" width="0.1524" layer="91"/>
+<label x="208.28" y="43.18" size="1.778" layer="95" rot="R90"/>
+</segment>
+</net>
